File: IPCMemoryExpansionBoard/IPCMemoryExpansionBoard.sch (KiCad schematic (older format))
At the start: 66 parts, among them J1 C64AC, J2 Micro_SD_Card_Det_Hirose_DM3AT, J3 USB_B_Mini, J4 JTAG, J5 JTAG-STM32, J6 SERIAL, SW1 SW_DIP_x08, U1 74LVC245, U10 74LVC245, U11 74LS38, U12 74LS38, U13 AMS1117-3.3, U2 74LVC245, U3 74LVC245, U4 74LVC245, U5 74LVC245, U6 XC2C32A, U7 SST38VF6401, U8 AS6C6416, U9 STM32F407ZETx, Y1 8MHz

Commit message: Updates and fixes.
Parts:
- removed J3: USB_B_Mini, symbol Connector:USB_B_Mini
- removed R14: 1.5k, symbol Device:R_Small
- added C27, C28, C29, C30, C31, C32: 100n, Capacitor_SMD:C_0805_2012Metric_Pad1.15x1.40mm_HandSolder, symbol Device:C_Small
- added J3: USB_B_Micro, Connector_USB:USB_Micro-B_Wuerth_614105150721_Vertical, symbol Connector:USB_B_Micro
- added J7: 6P6C, Connector_RJ:RJ12_Amphenol_54601, symbol Connector:6P6C
- added unit 5 of U11
- C1, C2, C3, C5, C6, C8: footprint (none) -> Capacitor_THT:C_Disc_D4.3mm_W1.9mm_P5.00mm
- C10, C4: footprint (none) -> Capacitor_THT:CP_Radial_D5.0mm_P2.50mm
- C11, C12, C13, C14, C15, C16, C17, C18, C19, C20, C21, C22, C23, C24, C25, C26, C9: footprint (none) -> Capacitor_SMD:C_0805_2012Metric_Pad1.15x1.40mm_HandSolder
- C7: value C_Small -> 100n; footprint (none) -> Capacitor_THT:C_Disc_D4.3mm_W1.9mm_P5.00mm
- D1: value D_Small_ALT -> 1N4148; footprint (none) -> Diode_SMD:D_SOD-123
- D2, D3, D4: footprint (none) -> LED_THT:LED_D5.0mm_Horizontal_O1.27mm_Z3.0mm
- J1: footprint (none) -> kicadlibs:DIN41612_C_2x32_Male_Horizontal_THT
- J2: footprint (none) -> Connector_Card:microSD_HC_Hirose_DM3AT-SF-PEJM5
- J4: footprint (none) -> Connector_IDC:IDC-Header_2x07_P2.54mm_Horizontal
- J5: footprint (none) -> Connector_IDC:IDC-Header_2x10_P2.54mm_Horizontal
- J6: footprint (none) -> Connector_PinHeader_2.54mm:PinHeader_1x03_P2.54mm_Horizontal
- R1: value R_Small -> 10k; footprint (none) -> Resistor_SMD:R_0805_2012Metric_Pad1.15x1.40mm_HandSolder
- R10, R11, R12, R13, R15, R2, R3, R4, R5, R6, R7, R8, R9: footprint (none) -> Resistor_SMD:R_0805_2012Metric_Pad1.15x1.40mm_HandSolder
- SW1: footprint (none) -> Package_DIP:DIP-16_W7.62mm
- U1, U10, U2, U3, U4, U5: footprint (none) -> Package_DIP:DIP-20_W7.62mm
- U11: renamed from U12; footprint (none) -> Package_DIP:DIP-14_W7.62mm
- U11: footprint (none) -> Package_DIP:DIP-14_W7.62mm
- U6: footprint (none) -> Package_QFP:TQFP-44_10x10mm_P0.8mm
- U7, U8: footprint (none) -> Package_SO:TSOP-I-48_18.4x12mm_P0.5mm
- Y1: footprint (none) -> Crystal:Crystal_HC49-U_Vertical
Connections:
- net labels added: SCL, SDA
- wire segments 657 -> 672
- no-connect marks 72 -> 73

Commit message: Update schematic. Fixed PCB. Added zip for gerbers.
Parts:
- added D5, D6: MBRS130L, Diode_SMD:D_SMB_Handsoldering, symbol Device:D_Schottky_Small
- added R14: 10k, Resistor_SMD:R_0805_2012Metric_Pad1.15x1.40mm_HandSolder, symbol IPCMemoryExpansionBoard-rescue:R_Small-Device
- C1, C11, C12, C13, C14, C15, C16, C17, C18, C19, C2, C20, C21, C22, C23, C24, C25, C26, C27, C28, C29, C3, C30, C31, C32, C5, C6, C7, C8, C9: symbol Device:C_Small -> IPCMemoryExpansionBoard-rescue:C_Small-Device
- C10, C4: symbol Device:CP_Small -> IPCMemoryExpansionBoard-rescue:CP_Small-Device
- D1: symbol Device:D_Small_ALT -> IPCMemoryExpansionBoard-rescue:D_Small_ALT-Device
- D2, D3, D4: footprint LED_THT:LED_D5.0mm_Horizontal_O1.27mm_Z3.0mm -> LED_THT:LED_D3.0mm_Horizontal_O1.27mm_Z2.0mm; symbol Device:LED_ALT -> IPCMemoryExpansionBoard-rescue:LED_ALT-Device
- J1: symbol Connector:C64AC -> IPCMemoryExpansionBoard-rescue:C64AC-Connector
- J2: symbol Connector:Micro_SD_Card_Det_Hirose_DM3AT -> IPCMemoryExpansionBoard-rescue:Micro_SD_Card_Det_Hirose_DM3AT-Connector
- J3: footprint Connector_USB:USB_Micro-B_Wuerth_614105150721_Vertical -> Connector_USB:USB_Mini-B_Lumberg_2486_01_Horizontal; symbol Connector:USB_B_Micro -> IPCMemoryExpansionBoard-rescue:USB_B_Micro-Connector
- J4: symbol Connector_Generic:Conn_02x07_Odd_Even -> IPCMemoryExpansionBoard-rescue:Conn_02x07_Odd_Even-Connector_Generic
- J5: symbol Connector_Generic:Conn_02x10_Odd_Even -> IPCMemoryExpansionBoard-rescue:Conn_02x10_Odd_Even-Connector_Generic
- R1, R10, R11, R12, R13, R15, R2, R3, R4, R5, R6, R7, R8, R9: symbol Device:R_Small -> IPCMemoryExpansionBoard-rescue:R_Small-Device
- SW1: symbol Switch:SW_DIP_x08 -> IPCMemoryExpansionBoard-rescue:SW_DIP_x08-Switch
- U1, U10, U2, U3, U4, U5: symbol tinkerforge:74LVC245 -> IPCMemoryExpansionBoard-rescue:74LVC245-tinkerforge
- U11: symbol 74xx:74LS38 -> IPCMemoryExpansionBoard-rescue:74LS38-74xx
- U13: symbol Regulator_Linear:AMS1117-3.3 -> IPCMemoryExpansionBoard-rescue:AMS1117-3.3-Regulator_Linear
- U9: symbol MCU_ST_STM32F4:STM32F407ZETx -> IPCMemoryExpansionBoard-rescue:STM32F407ZETx-MCU_ST_STM32F4
- Y1: symbol Device:Crystal_Small -> IPCMemoryExpansionBoard-rescue:Crystal_Small-Device
Connections:
- wire segments 672 -> 689
- no-connect marks 73 -> 68
Other:
- moved on the sheet: C11, C8

Commit message: Small fixes to the PCB. RESET was short circuit to GND
Connections:
- wire segments 689 -> 687
Changed lines of the file:
@@
 	4550 4200 4850 4200
-Wire Wire Line
-	4550 4300 4600 4300
 Wire Wire Line
 	4550 4900 4850 4900
@@
 L IPCMemoryExpansionBoard-rescue:GND-power #PWR0120
 U 1 1 61044D61
-P 4600 4450
-F 0 "#PWR0120" H 4600 4200 50  0001 C CNN
-F 1 "GND" H 4605 4277 50  0000 C CNN
-F 2 "" H 4600 4450 50  0001 C CNN
-F 3 "" H 4600 4450 50  0001 C CNN
-	1    4600 4450
-	1    0    0    -1
-$EndComp
-Wire Wire Line
-	4550 3500 4600 3500
-Wire Wire Line
-	4600 3500 4600 4300
-Connection ~ 4600 4400
-Wire Wire Line
-	4600 4300 4850 4300
-Wire Wire Line
-	4600 4300 4600 4400
-Wire Wire Line
-	4550 4400 4600 4400
-Wire Wire Line
-	4600 4400 4600 4450
+P 5000 4450
+F 0 "#PWR0120" H 5000 4200 50  0001 C CNN
+F 1 "GND" H 5005 4277 50  0000 C CNN
+F 2 "" H 5000 4450 50  0001 C CNN
+F 3 "" H 5000 4450 50  0001 C CNN
+	1    5000 4450
+	1    0    0    -1
+$EndComp
+Wire Wire Line
+	4550 3500 5000 3500
+Wire Wire Line
+	5000 3500 5000 4400
+Connection ~ 5000 4400
+Wire Wire Line
+	4550 4400 5000 4400
+Wire Wire Line
+	5000 4400 5000 4450
 Text Label 3250 900  0    50   ~ 0
 OE245
@@
 Wire Wire Line
 	2050 1300 2100 1300
+Wire Wire Line
+	4550 4300 4850 4300
 $EndSCHEMATC

Commit message: Started work on spin 2.
Parts:
- removed J2: Micro_SD_Card_Det_Hirose_DM3AT, Connector_Card:microSD_HC_Hirose_DM3AT-SF-PEJM5, symbol IPCMemoryExpansionBoard-rescue:Micro_SD_Card_Det_Hirose_DM3AT-Connector
- removed J7: 6P6C, Connector_RJ:RJ12_Amphenol_54601, symbol Connector:6P6C
- added J10, J11, J12, J8, J9: TESTPOINTS, Connector_PinHeader_2.54mm:PinHeader_1x08_P2.54mm_Vertical, symbol Connector:Conn_01x08_Male
- added J13, J14, J15, J16, J17, J18, J19, J20, J21, J22, J23: TESTPOINT, Connector_PinHeader_2.54mm:PinHeader_1x01_P2.54mm_Vertical, symbol Connector:Conn_01x01_Male
- added J2: TESTPOINTS, Connector_PinHeader_2.54mm:PinHeader_1x05_P2.54mm_Vertical, symbol Connector:Conn_01x05_Male
- added J7: TESTPOINTS, Connector_PinHeader_2.54mm:PinHeader_1x02_P2.54mm_Vertical, symbol Connector:Conn_01x02_Male
- added RN1, RN15, RN16, RN2: Resistor net 56 ohm, Resistor_THT:R_Array_SIP8, symbol Device:R_Pack04_SIP
- added RN10: 3.3k, Resistor_THT:R_Array_SIP6, symbol Device:R_Network05
- added RN11, RN12, RN3, RN4, RN5: 3.9k, Resistor_THT:R_Array_SIP9, symbol Device:R_Network08
- added RN13, RN14, RN7, RN8, RN9: 3.3k, Resistor_THT:R_Array_SIP9, symbol Device:R_Network08
- added RN6: 3.9k, Resistor_THT:R_Array_SIP6, symbol Device:R_Network05
- SW1: value SW_DIP_x08 -> CONFIG SWITCH
Connections:
- net labels added: NAS, NBAS, RD0, RD1, RD10, RD11, RD12, RD13, RD14, RD15, RD2, RD3, RD4, RD5, RD6, RD7, RD8, RD9
- net labels removed: DIPSW6, DIPSW7, SCL, SDA, SDIO_CMD, SDIO_D0, SDIO_D1, SDIO_D2, SDIO_D3, SDIO_SCK
- wire segments 687 -> 755
- no-connect marks 68 -> 71
Other:
- moved on the sheet: C5, C7, D2, D3, D4, D6, J3, J5, R12, R13, R2, R3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

Commit message: Made spin 2 of the board
Parts:
- added J24, J25, J26, J27, J28, J29: TESTPOINT, Connector_PinHeader_2.54mm:PinHeader_1x01_P2.54mm_Vertical, symbol Connector:Conn_01x01_Male
Connections:
- net labels added: USB_N, USB_P
- net labels removed: USB_DM, USB_DP
- wire segments 755 -> 765
Changed lines of the file:
@@
 Text Label 1350 8700 0    50   ~ 0
 NBUD
-Text Label 1350 8500 0    50   ~ 0
-BRNW
 Text Label 1350 8300 0    50   ~ 0
+BRNW
+Text Label 1350 8400 0    50   ~ 0
 BNPS
 Text Label 2500 8500 0    50   ~ 0
@@
 Text Label 2500 8600 0    50   ~ 0
 NUD
-Text Label 2500 8400 0    50   ~ 0
-RNW
 Text Label 2500 8200 0    50   ~ 0
+RNW
+Text Label 2500 8300 0    50   ~ 0
 NPS
 $Comp
@@
 	10700 10450 11500 10450
 Text Label 11250 10350 0    50   ~ 0
-USB_DP
+USB_P
 Text Label 11250 10450 0    50   ~ 0
-USB_DM
+USB_N
 $Comp
 L IPCMemoryExpansionBoard-rescue:R_Small-Device R15
@@
 	14300 2250 14900 2250
 Text Label 14450 2250 0    50   ~ 0
-USB_DM
+USB_N
 Text Label 14450 2350 0    50   ~ 0
-USB_DP
+USB_P
 Wire Wire Line
 	11900 4150 11450 4150
@@
 Wire Wire Line
 	1300 8700 1700 8700
-Text Label 1350 8400 0    50   ~ 0
+Text Label 1350 8500 0    50   ~ 0
 NBAS
 Wire Wire Line
 	2400 8600 2800 8600
-Text Label 2500 8300 0    50   ~ 0
+Text Label 2500 8400 0    50   ~ 0
 NAS
 Wire Wire Line
@@
 Wire Wire Line
 	4300 6900 3800 6900
-Text Label 3950 6500 0    50   ~ 0
+Text Label 3950 6600 0    50   ~ 0
 BNPS
-Text Label 3950 6700 0    50   ~ 0
+Text Label 3950 6500 0    50   ~ 0
 BRNW
-Text Label 3950 6600 0    50   ~ 0
+Text Label 3950 6700 0    50   ~ 0
 NBAS
 Text Label 3950 6900 0    50   ~ 0
@@
 Text Label 3150 7750 0    50   ~ 0
 NBUD
-Text Label 3150 7450 0    50   ~ 0
-NBAS
 Text Label 3150 7550 0    50   ~ 0
-BRNW
+NBAS
 Text Label 3150 7350 0    50   ~ 0
+BRNW
+Text Label 3150 7450 0    50   ~ 0
 BNPS
 $Comp
@@
 	3850 7300 4150 7300
 Text Label 3900 7200 0    50   ~ 0
-NBDTACK
+DTACK
 Text Label 3900 7300 0    50   ~ 0
-NBIMA
+IMA
 $Comp
 L IPCMemoryExpansionBoard-rescue:GND-power #PWR0105
@@
 Wire Wire Line
 	4800 6950 4800 6900
+$Comp
+L Connector:Conn_01x01_Male J28
+U 1 1 61D14167
+P 8900 9400
+F 0 "J28" H 9006 9578 50  0000 C CNN
+F 1 "TESTPOINT" H 9006 9487 50  0000 C CNN
+F 2 "Connector_PinHeader_2.54mm:PinHeader_1x01_P2.54mm_Vertical" H 8900 9400 50  0001 C CNN
+F 3 "~" H 8900 9400 50  0001 C CNN
+	1    8900 9400
+	1    0    0    -1
+$EndComp
+$Comp
+L Connector:Conn_01x01_Male J27
+U 1 1 61D1465E
+P 8900 9150
+F 0 "J27" H 9006 9328 50  0000 C CNN
+F 1 "TESTPOINT" H 9006 9237 50  0000 C CNN
+F 2 "Connector_PinHeader_2.54mm:PinHeader_1x01_P2.54mm_Vertical" H 8900 9150 50  0001 C CNN
+F 3 "~" H 8900 9150 50  0001 C CNN
+	1    8900 9150
+	1    0    0    -1
+$EndComp
+$Comp
+L Connector:Conn_01x01_Male J26
+U 1 1 61DF0FDD
+P 8900 8900
+F 0 "J26" H 9006 9078 50  0000 C CNN
+F 1 "TESTPOINT" H 9006 8987 50  0000 C CNN
+F 2 "Connector_PinHeader_2.54mm:PinHeader_1x01_P2.54mm_Vertical" H 8900 8900 50  0001 C CNN
+F 3 "~" H 8900 8900 50  0001 C CNN
+	1    8900 8900
+	1    0    0    -1
+$EndComp
+$Comp
+L Connector:Conn_01x01_Male J25
+U 1 1 61DF1170
+P 8900 8650
+F 0 "J25" H 9006 8828 50  0000 C CNN
+F 1 "TESTPOINT" H 9006 8737 50  0000 C CNN
+F 2 "Connector_PinHeader_2.54mm:PinHeader_1x01_P2.54mm_Vertical" H 8900 8650 50  0001 C CNN
+F 3 "~" H 8900 8650 50  0001 C CNN
+	1    8900 8650
+	1    0    0    -1
+$EndComp
+$Comp
+L IPCMemoryExpansionBoard-rescue:GND-power #PWR0104
+U 1 1 61DF127E
+P 9350 9550
+F 0 "#PWR0104" H 9350 9300 50  0001 C CNN
+F 1 "GND" H 9355 9377 50  0000 C CNN
+F 2 "" H 9350 9550 50  0001 C CNN
+F 3 "" H 9350 9550 50  0001 C CNN
+	1    9350 9550
+	1    0    0    -1
+$EndComp
+Wire Wire Line
+	9350 9550 9350 9400
+Wire Wire Line
+	9350 8650 9100 8650
+Wire Wire Line
+	9100 8900 9350 8900
+Connection ~ 9350 8900
+Wire Wire Line
+	9350 8900 9350 8650
+Wire Wire Line
+	9100 9150 9350 9150
+Connection ~ 9350 9150
+Wire Wire Line
+	9350 9150 9350 8900
+Wire Wire Line
+	9100 9400 9350 9400
+Connection ~ 9350 9400
+Wire Wire Line
+	9350 9400 9350 9150
+$Comp
+L Connector:Conn_01x01_Male J24
+U 1 1 6216A69B
+P 7550 10300
+F 0 "J24" H 7656 10478 50  0000 C CNN
+F 1 "TESTPOINT" H 7656 10387 50  0000 C CNN
+F 2 "Connector_PinHeader_2.54mm:PinHeader_1x01_P2.54mm_Vertical" H 7550 10300 50  0001 C CNN
+F 3 "~" H 7550 10300 50  0001 C CNN
+	1    7550 10300
+	1    0    0    -1
+$EndComp
+$Comp
+L Connector:Conn_01x01_Male J29
+U 1 1 6216AAFF
+P 9550 10300
+F 0 "J29" H 9550 10400 50  0000 C CNN
+F 1 "TESTPOINT" H 9600 10200 50  0000 C CNN
+F 2 "Connector_PinHeader_2.54mm:PinHeader_1x01_P2.54mm_Vertical" H 9550 10300 50  0001 C CNN
+F 3 "~" H 9550 10300 50  0001 C CNN
+	1    9550 10300
+	-1   0    0    1
+$EndComp
+Wire Wire Line
+	9350 10300 9150 10300
+Wire Wire Line
+	7750 10300 7950 10300
 $EndSCHEMATC
