File: IPCMemoryExpansionBoard/IPCMemoryExpansionBoard.kicad_pcb (KiCad board)
At the start: 2 copper layers, 71 parts, among them J1 C64AC, J2 Micro_SD_Card_Det_Hirose_DM3AT, J3 USB_B_Micro, J4 JTAG, J5 JTAG-STM32, J6 SERIAL, J7 6P6C, SW1 SW_DIP_x08, U1 74LVC245, U10 74LVC245, U11 74LS38, U13 AMS1117-3.3, U2 74LVC245, U3 74LVC245, U4 74LVC245, U5 74LVC245, U6 XC2C32A, U7 SST38VF6401, U8 AS6C6416, U9 STM32F407ZETx, Y1 8MHz

Commit message: Update schematic. Fixed PCB. Added zip for gerbers.
Parts:
- added D5: MBRS130L, Diode_SMD:D_SMB_Handsoldering, F.Cu at (73.8, 40.9)
- added D6: MBRS130L, Diode_SMD:D_SMB_Handsoldering, F.Cu at (34.9, 130.2)
- added R14: 10k, Resistor_SMD:R_0805_2012Metric_Pad1.15x1.40mm_HandSolder, B.Cu at (205.7, 63.2)
- C11, C12, C13, C14, C15, C16, C17, C18, C19, C20, C21, C23, C24, C25, C26, C27, C28, C29, C30, C31, C32, C9, R10, R2, R3, R4, R5, R6, R7, R8, R9, U13: moved to B.Cu
- D2, D3, D4: footprint LED_THT:LED_D5.0mm_Horizontal_O1.27mm_Z3.0mm -> LED_THT:LED_D3.0mm_Horizontal_O1.27mm_Z2.0mm
- J3: footprint Connector_USB:USB_Micro-B_Wuerth_614105150721_Vertical -> Connector_USB:USB_Mini-B_Lumberg_2486_01_Horizontal
- moved C9 186.4 mm to (40.0, 99.7)
- moved C10 176.1 mm to (39.7, 37.8), turned to 90 degrees
- moved J7 163.5 mm to (44.1, 128.7)
- moved C28 163.1 mm to (56.0, 98.5)
- moved U8 160.6 mm to (39.8, 99.9), turned to 270 degrees
- moved C4 157.2 mm to (60.5, 38.7), turned to 90 degrees
- moved R5 155.8 mm to (83.2, 139.8), turned to 270 degrees
- moved D2 155.0 mm to (111.6, 139.1)
- moved D4 153.5 mm to (106.7, 139.1)
- moved R6 146.0 mm to (89.9, 139.6), turned to 270 degrees
- moved R7 145.4 mm to (92.7, 139.6), turned to 270 degrees
- moved R8 145.3 mm to (87.4, 139.6), turned to 90 degrees
- moved C5 145.1 mm to (35.6, 61.7), turned to 270 degrees
- moved C30 134.4 mm to (98.4, 138.6), turned to 180 degrees
- moved R9 134.1 mm to (95.0, 139.6), turned to 270 degrees
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Connections:
- C8 pad 1: +3V3 -> +5V
- J1 pad A24: (no net) -> Net-(J1-PadA24)
- J1 pad A27: (no net) -> Net-(J1-PadA27)
- J1 pad A29: (no net) -> Net-(J1-PadA29)
- J1 pad A30: (no net) -> Net-(J1-PadA30)
- J1 pad A32: (no net) -> Net-(J1-PadA32)
- J1 pad C1: (no net) -> Net-(J1-PadC1)
- J1 pad C2: +5V -> Net-(D5-Pad2)
- J1 pad C23: (no net) -> Net-(J1-PadC23)
- J1 pad C25: (no net) -> Net-(J1-PadC25)
- J1 pad C27: (no net) -> Net-(J1-PadC27)
- J1 pad C29: (no net) -> Net-(J1-PadC29)
- J1 pad C30: (no net) -> Net-(J1-PadC30)
- J1 pad C31: +5V -> Net-(D5-Pad2)
- J2 pad 10: (no net) -> Net-(J2-Pad10)
- J2 pad 9: (no net) -> Net-(J2-Pad9)
- J3 pad 1: +5V -> Net-(D6-Pad2)
- J3 pad 4: (no net) -> Net-(J3-Pad4)
- J4 pad 12: (no net) -> Net-(J4-Pad12)
- J4 pad 14: (no net) -> Net-(J4-Pad14)
- J5 pad 11: (no net) -> Net-(J5-Pad11)
- J5 pad 17: (no net) -> Net-(J5-Pad17)
- J5 pad 19: (no net) -> Net-(J5-Pad19)
- J7 pad 1: (no net) -> Net-(J7-Pad1)
- J7 pad 6: (no net) -> Net-(J7-Pad6)
- U10 pad 11: (no net) -> Net-(R14-Pad1)
- U10 pad 12: (no net) -> Net-(R14-Pad1)
- U10 pad 13: (no net) -> Net-(R14-Pad1)
- U10 pad 14: (no net) -> Net-(R14-Pad1)
- U10 pad 15: /BNPS -> /NBUD
- U10 pad 16: /BRNW -> /NBLD
- U10 pad 17: /NBUD -> /BRNW
- U10 pad 18: /NBLD -> /BNPS
- U10 pad 2: /NLD -> /NPS
- U10 pad 3: /NUD -> /RNW
- U10 pad 4: /RNW -> /NLD
- U10 pad 5: /NPS -> /NUD
- U10 pad 6: (no net) -> Net-(U10-Pad6)
- U10 pad 7: (no net) -> Net-(U10-Pad7)
- U10 pad 8: (no net) -> Net-(U10-Pad8)
- U10 pad 9: (no net) -> Net-(U10-Pad9)
- U11 pad 14: GND -> +5V
- U11 pad 7: +5V -> GND
- U4 pad 11: /D7 -> /BD7
- U4 pad 12: /D6 -> /BD6
- U4 pad 13: /D5 -> /BD5
- U4 pad 14: /D4 -> /BD4
- U4 pad 15: /D3 -> /BD3
- U4 pad 16: /D2 -> /BD2
- U4 pad 17: /D1 -> /BD1
- U4 pad 18: /D0 -> /BD0
- U4 pad 2: /BD0 -> /D0
- U4 pad 3: /BD1 -> /D1
- U4 pad 4: /BD2 -> /D2
- U4 pad 5: /BD3 -> /D3
- U4 pad 6: /BD4 -> /D4
- U4 pad 7: /BD5 -> /D5
- U4 pad 8: /BD6 -> /D6
- U4 pad 9: /BD7 -> /D7
- U5 pad 11: /D15 -> /BD15
- U5 pad 12: /D14 -> /BD14
- U5 pad 13: /D13 -> /BD13
- U5 pad 14: /D12 -> /BD12
- U5 pad 15: /D11 -> /BD11
- U5 pad 16: /D10 -> /BD10
- U5 pad 17: /D9 -> /BD9
- U5 pad 18: /D8 -> /BD8
- U5 pad 2: /BD8 -> /D8
- U5 pad 3: /BD9 -> /D9
- U5 pad 4: /BD10 -> /D10
- U5 pad 5: /BD11 -> /D11
- U5 pad 6: /BD12 -> /D12
- U5 pad 7: /BD13 -> /D13
- U5 pad 8: /BD14 -> /D14
- U5 pad 9: /BD15 -> /D15
- U9 pad 1: (no net) -> Net-(U9-Pad1)
- U9 pad 100: (no net) -> Net-(U9-Pad100)
- U9 pad 117: (no net) -> Net-(U9-Pad117)
- U9 pad 122: (no net) -> Net-(U9-Pad122)
- U9 pad 123: (no net) -> Net-(U9-Pad123)
- U9 pad 129: (no net) -> Net-(U9-Pad129)
- U9 pad 132: (no net) -> Net-(U9-Pad132)
- U9 pad 135: (no net) -> Net-(U9-Pad135)
- U9 pad 136: (no net) -> Net-(U9-Pad136)
- U9 pad 137: (no net) -> Net-(U9-Pad137)
- U9 pad 139: (no net) -> Net-(U9-Pad139)
- U9 pad 140: (no net) -> Net-(U9-Pad140)
- U9 pad 18: (no net) -> Net-(U9-Pad18)
- U9 pad 19: (no net) -> Net-(U9-Pad19)
- U9 pad 20: (no net) -> Net-(U9-Pad20)
- U9 pad 21: (no net) -> Net-(U9-Pad21)
- U9 pad 22: (no net) -> Net-(U9-Pad22)
- U9 pad 26: (no net) -> Net-(U9-Pad26)
- U9 pad 27: (no net) -> Net-(U9-Pad27)
- U9 pad 28: (no net) -> Net-(U9-Pad28)
- U9 pad 29: (no net) -> Net-(U9-Pad29)
- U9 pad 34: (no net) -> Net-(U9-Pad34)
- U9 pad 35: (no net) -> Net-(U9-Pad35)
- U9 pad 36: (no net) -> Net-(U9-Pad36)
- U9 pad 37: (no net) -> Net-(U9-Pad37)
- U9 pad 40: (no net) -> Net-(U9-Pad40)
- U9 pad 41: (no net) -> Net-(U9-Pad41)
- U9 pad 42: (no net) -> Net-(U9-Pad42)
- U9 pad 43: (no net) -> Net-(U9-Pad43)
- U9 pad 44: (no net) -> Net-(U9-Pad44)
- U9 pad 45: (no net) -> Net-(U9-Pad45)
- U9 pad 46: (no net) -> Net-(U9-Pad46)
- U9 pad 47: (no net) -> Net-(U9-Pad47)
- U9 pad 49: (no net) -> Net-(U9-Pad49)
- U9 pad 7: (no net) -> Net-(U9-Pad7)
- U9 pad 73: (no net) -> Net-(U9-Pad73)
- U9 pad 74: (no net) -> Net-(U9-Pad74)
- U9 pad 75: (no net) -> Net-(U9-Pad75)
- U9 pad 76: (no net) -> Net-(U9-Pad76)
- U9 pad 8: (no net) -> Net-(U9-Pad8)
- U9 pad 9: (no net) -> Net-(U9-Pad9)
- U9 pad 96: (no net) -> Net-(U9-Pad96)
- U9 pad 97: (no net) -> Net-(U9-Pad97)
Routing:
- net GND: track 0.00 -> 1144.0 mm, vias 0 -> 36
- net +3V3: track 0.00 -> 737.8 mm, vias 0 -> 32
- net /D1: track 0.00 -> 271.0 mm, vias 0 -> 9
- net /D0: track 0.00 -> 269.5 mm, vias 0 -> 9
- net +5V: track 0.00 -> 265.5 mm, vias 0 -> 1
- net /NLD: track 0.00 -> 262.9 mm, vias 0 -> 9
- net /NUD: track 0.00 -> 261.7 mm, vias 0 -> 10
- net /D7: track 0.00 -> 249.7 mm, vias 0 -> 9
- net /D15: track 0.00 -> 240.5 mm, vias 0 -> 7
- net /D14: track 0.00 -> 236.5 mm, vias 0 -> 7
- net /D3: track 0.00 -> 234.4 mm, vias 0 -> 9
- net /D2: track 0.00 -> 232.3 mm, vias 0 -> 9
- net /D13: track 0.00 -> 231.8 mm, vias 0 -> 7
- net /ROMADR2: track 0.00 -> 230.1 mm, vias 0 -> 10
- net /ROMADR1: track 0.00 -> 227.9 mm, vias 0 -> 7
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- added copper zone on B.Cu, net +3V3
- added copper zone on F.Cu, net GND
Other:
- board outline added: 185 x 116 mm
- net class PWR added: clearance 0.2, trace_width 0.25, via_dia 0.8, via_drill 0.4
- board text added: "GND"
- board text added: "HP IPC Memory Expansion board."
- board text added: "I2C and +5V"
- board text added: "JTAG STM32"
- board text added: "JTAG Xilinx"
- board text added: "Mattis Lind 2021 www.datormuseum.se"
- board text added: "RX"
- board text added: "Serial 3.3V levels"
- board text added: "TX"
- board text added: "https://github.com/MattisLind/IPCMemoryExpansion"

Commit message: Started work on spin 2.
Parts:
- added J10: TESTPOINTS, Connector_PinHeader_2.54mm:PinHeader_1x08_P2.54mm_Vertical, F.Cu at (104.1, 52.7)
- added J11: TESTPOINTS, Connector_PinHeader_2.54mm:PinHeader_1x08_P2.54mm_Vertical, F.Cu at (133.3, 52.7)
- added J12: TESTPOINTS, Connector_PinHeader_2.54mm:PinHeader_1x08_P2.54mm_Vertical, F.Cu at (162.6, 52.7)
- added J13: TESTPOINT, Connector_PinHeader_2.54mm:PinHeader_1x01_P2.54mm_Vertical, F.Cu at (222.8, 98.8)
- added J14: TESTPOINT, Connector_PinHeader_2.54mm:PinHeader_1x01_P2.54mm_Vertical, F.Cu at (226.5, 98.8)
- added J15: TESTPOINT, Connector_PinHeader_2.54mm:PinHeader_1x01_P2.54mm_Vertical, F.Cu at (239.0, 92.1)
- added J16: TESTPOINT, Connector_PinHeader_2.54mm:PinHeader_1x01_P2.54mm_Vertical, F.Cu at (233.8, 98.8)
- added J17: TESTPOINT, Connector_PinHeader_2.54mm:PinHeader_1x01_P2.54mm_Vertical, F.Cu at (222.8, 102.5)
- added J18: TESTPOINT, Connector_PinHeader_2.54mm:PinHeader_1x01_P2.54mm_Vertical, F.Cu at (226.5, 102.5)
- added J19: TESTPOINT, Connector_PinHeader_2.54mm:PinHeader_1x01_P2.54mm_Vertical, F.Cu at (182.9, 113.0)
- added J20: TESTPOINT, Connector_PinHeader_2.54mm:PinHeader_1x01_P2.54mm_Vertical, F.Cu at (261.2, 72.0)
- added J21: TESTPOINT, Connector_PinHeader_2.54mm:PinHeader_1x01_P2.54mm_Vertical, F.Cu at (242.6, 92.1)
- added J22: TESTPOINT, Connector_PinHeader_2.54mm:PinHeader_1x01_P2.54mm_Vertical, F.Cu at (239.0, 95.8)
- added J23: TESTPOINT, Connector_PinHeader_2.54mm:PinHeader_1x01_P2.54mm_Vertical, F.Cu at (230.1, 98.8)
- added J8: TESTPOINTS, Connector_PinHeader_2.54mm:PinHeader_1x08_P2.54mm_Vertical, F.Cu at (44.5, 52.7)
- added J9: TESTPOINTS, Connector_PinHeader_2.54mm:PinHeader_1x08_P2.54mm_Vertical, F.Cu at (74.9, 52.7)
- added RN1: R_Pack04_SIP, Resistor_THT:R_Array_SIP8, F.Cu at (133.3, 50.2)
- added RN10: R_Network05, Resistor_THT:R_Array_SIP6, F.Cu at (204.5, 57.8)
- added RN11: R_Network08, Resistor_THT:R_Array_SIP9, F.Cu at (130.8, 57.8)
- added RN12: R_Network08, Resistor_THT:R_Array_SIP9, F.Cu at (160.0, 57.8)
- added RN13: R_Network08, Resistor_THT:R_Array_SIP9, F.Cu at (130.8, 55.2)
- added RN14: R_Network08, Resistor_THT:R_Array_SIP9, F.Cu at (160.0, 55.2)
- added RN15: R_Pack04_SIP, Resistor_THT:R_Array_SIP8, F.Cu at (162.6, 50.2)
- added RN16: R_Pack04_SIP, Resistor_THT:R_Array_SIP8, F.Cu at (162.6, 47.6)
- added RN2: R_Pack04_SIP, Resistor_THT:R_Array_SIP8, F.Cu at (133.3, 47.6)
- added RN3: R_Network08, Resistor_THT:R_Array_SIP9, F.Cu at (41.9, 57.8)
- added RN4: R_Network08, Resistor_THT:R_Array_SIP9, F.Cu at (72.4, 57.8)
- added RN5: R_Network08, Resistor_THT:R_Array_SIP9, F.Cu at (101.6, 57.8)
- added RN6: R_Network05, Resistor_THT:R_Array_SIP6, F.Cu at (189.2, 55.2)
- added RN7: R_Network08, Resistor_THT:R_Array_SIP9, F.Cu at (41.9, 55.2)
- added RN8: R_Network08, Resistor_THT:R_Array_SIP9, F.Cu at (72.4, 55.2)
- added RN9: R_Network08, Resistor_THT:R_Array_SIP9, F.Cu at (101.6, 55.2)
- J2: value Micro_SD_Card_Det_Hirose_DM3AT -> TESTPOINTS; footprint Connector_Card:microSD_HC_Hirose_DM3AT-SF-PEJM5 -> Connector_PinHeader_2.54mm:PinHeader_1x05_P2.54mm_Vertical
- J7: value 6P6C -> TESTPOINTS; footprint Connector_RJ:RJ12_Amphenol_54601 -> Connector_PinHeader_2.54mm:PinHeader_1x02_P2.54mm_Vertical
- moved J7 176.5 mm to (201.2, 48.2), turned to 270 degrees
- moved J2 97.9 mm to (191.8, 52.7), turned to 90 degrees
- moved C8 29.4 mm to (209.1, 37.8)
- moved U11 8.16 mm to (191.0, 45.4)
- moved J6 7.78 mm to (149.2, 135.0)
- moved SW1 4.93 mm to (157.5, 144.1)
- moved J4 3.32 mm to (201.7, 132.4)
Connections:
- D1 pad 1: GND -> /NRESET
- J1 pad C25: Net-(J1-PadC25) -> /NBAS
- J2 pad 1: /SDIO_D2 -> /BNPS
- J2 pad 2: /SDIO_D3 -> /NBAS
- J2 pad 3: /SDIO_CMD -> /BRNW
- J2 pad 4: +3V3 -> /NBLD
- J2 pad 5: /SDIO_SCK -> /NBUD
- J7 pad 1: Net-(J7-Pad1) -> /NBDTACK
- J7 pad 2: GND -> /NBIMA
- SW1 pad 10: /DIPSW6 -> /STM32_RESET
- SW1 pad 9: /DIPSW7 -> /STM32_BUSEN
- U1 pad 19: /OE245 -> /STM32_BUSEN
- U1 pad 9: GND -> /NRESET
- U10 pad 14: Net-(R14-Pad1) -> /NBUD
- U10 pad 15: /NBUD -> /NBLD
- U10 pad 16: /NBLD -> /BRNW
- U10 pad 17: /BRNW -> /NBAS
- U10 pad 19: GND -> /STM32_BUSEN
- U10 pad 3: /RNW -> /NAS
- U10 pad 4: /NLD -> /RNW
- U10 pad 5: /NUD -> /NLD
- U10 pad 6: Net-(U10-Pad6) -> /NUD
- U2 pad 19: /OE245 -> /STM32_BUSEN
- U3 pad 16: /BA10 -> /BA11
- U3 pad 17: /BA11 -> /BA10
- U3 pad 19: /OE245 -> /STM32_BUSEN
- U4 pad 11: /BD7 -> /RD7
- U4 pad 12: /BD6 -> /RD6
- U4 pad 13: /BD5 -> /RD5
- U4 pad 14: /BD4 -> /RD4
- U4 pad 15: /BD3 -> /RD3
- U4 pad 16: /BD2 -> /RD2
- U4 pad 17: /BD1 -> /RD1
- U4 pad 18: /BD0 -> /RD0
- U5 pad 11: /BD15 -> /RD15
- U5 pad 12: /BD14 -> /RD14
- U5 pad 13: /BD13 -> /RD13
- U5 pad 14: /BD12 -> /RD12
- U5 pad 15: /BD11 -> /RD11
- U5 pad 16: /BD10 -> /RD10
- U5 pad 17: /BD9 -> /RD9
- U5 pad 18: /BD8 -> /RD8
- U6 pad 13: /NLD -> /NAS
- U6 pad 16: /NUD -> /D6
- U7 pad 12: GND -> /NRESET
- U9 pad 111: /SDIO_D2 -> Net-(U9-Pad111)
- U9 pad 112: /SDIO_D3 -> Net-(U9-Pad112)
- U9 pad 113: /SDIO_SCK -> Net-(U9-Pad113)
- U9 pad 116: /SDIO_CMD -> Net-(U9-Pad116)
- U9 pad 122: Net-(U9-Pad122) -> /FLASH_RY
- U9 pad 124: /DIPSW6 -> Net-(U9-Pad124)
- U9 pad 126: /DIPSW7 -> Net-(U9-Pad126)
- U9 pad 69: /SCL -> Net-(U9-Pad69)
- U9 pad 70: /SDA -> Net-(U9-Pad70)
- U9 pad 98: /SDIO_D0 -> Net-(U9-Pad98)
- U9 pad 99: /SDIO_D1 -> Net-(U9-Pad99)
Routing:
- net GND: track 1144.0 -> 959.6 mm, vias 36 -> 32
- net /OE245: track 192.5 -> 99.8 mm
- net /DIPSW7: track 81.2 -> 0.00 mm, vias 5 -> 0
- net /DIPSW6: track 77.1 -> 0.00 mm, vias 5 -> 0
- net Net-(D5-Pad2): track 86.1 -> 10.6 mm
- net /SCL: track 74.5 -> 0.00 mm, vias 3 -> 0
- net /SDA: track 74.3 -> 0.00 mm, vias 3 -> 0
- net /NBAS: track 0.00 -> 63.1 mm
- net /STM32_BUSEN: track 59.0 -> 120.5 mm
- net +3V3: track 737.8 -> 685.3 mm, vias 32 -> 31
- net /NBDTACK: track 50.5 -> 4.42 mm
- net +5V: track 265.5 -> 309.2 mm
- net /TCK: track 46.5 -> 5.41 mm
- net /DIPSW3: track 52.8 -> 12.5 mm
- net /TMS: track 47.8 -> 8.21 mm
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- removed copper zone on B.Cu, net +3V3
- removed copper zone on F.Cu, net GND

Commit message: Made spin 2 of the board
Parts:
- added J24: TESTPOINT, Connector_PinHeader_2.54mm:PinHeader_1x01_P2.54mm_Vertical, F.Cu at (95.8, 56.6)
- added J25: TESTPOINT, Connector_PinHeader_2.54mm:PinHeader_1x01_P2.54mm_Vertical, F.Cu at (205.2, 71.1)
- added J26: TESTPOINT, Connector_PinHeader_2.54mm:PinHeader_1x01_P2.54mm_Vertical, F.Cu at (125.5, 52.6)
- added J27: TESTPOINT, Connector_PinHeader_2.54mm:PinHeader_1x01_P2.54mm_Vertical, F.Cu at (156.0, 52.8)
- added J28: TESTPOINT, Connector_PinHeader_2.54mm:PinHeader_1x01_P2.54mm_Vertical, F.Cu at (66.5, 54.1)
- added J29: TESTPOINT, Connector_PinHeader_2.54mm:PinHeader_1x01_P2.54mm_Vertical, F.Cu at (205.7, 101.3)
- RN1, RN15, RN16, RN2: value R_Pack04_SIP -> Resistor net 56 ohm
- RN10: value R_Network05 -> 3.3k
- RN11, RN12, RN3, RN4, RN5: value R_Network08 -> 3.9k
- RN13, RN14, RN7, RN8, RN9: value R_Network08 -> 3.3k
- RN6: value R_Network05 -> 3.9k
- SW1: value SW_DIP_x08 -> CONFIG SWITCH
- moved J20 82.0 mm to (189.1, 111.0)
- moved J23 73.4 mm to (156.8, 101.5)
- moved J22 56.2 mm to (183.2, 102.8)
- moved J14 54.7 mm to (172.7, 88.8)
- moved J13 54.6 mm to (169.5, 87.2)
- moved J15 54.1 mm to (186.1, 80.6)
- moved J21 48.8 mm to (195.1, 80.7)
- moved J16 37.8 mm to (198.1, 86.4)
- moved J18 35.6 mm to (191.8, 110.7)
- moved J17 27.9 mm to (201.3, 84.7)
- moved J19 12.7 mm to (170.7, 109.3)
Connections:
- net /USB_DM renamed /USB_N
- net /USB_DP renamed /USB_P
- J2 pad 1: /BNPS -> /BRNW
- J2 pad 2: /NBAS -> /BNPS
- J2 pad 3: /BRNW -> /NBAS
- J7 pad 1: /NBDTACK -> /DTACK
- J7 pad 2: /NBIMA -> /IMA
- RN10 pad 4: /BRNW -> /NBAS
- RN10 pad 5: /NBAS -> /BNPS
- RN10 pad 6: /BNPS -> /BRNW
- RN6 pad 2: /BNPS -> /BRNW
- RN6 pad 3: /NBAS -> /BNPS
- RN6 pad 4: /BRNW -> /NBAS
- U10 pad 16: /BRNW -> /NBAS
- U10 pad 17: /NBAS -> /BNPS
- U10 pad 18: /BNPS -> /BRNW
- U10 pad 2: /NPS -> /RNW
- U10 pad 3: /NAS -> /NPS
- U10 pad 4: /RNW -> /NAS
Routing:
- net GND: track 959.6 -> 1166.6 mm, vias 32 -> 33
- net /STM32_BUSEN: track 120.5 -> 283.5 mm, vias 2 -> 9
- net +5V: track 309.2 -> 432.8 mm, vias 1 -> 4
- net /STM32_RESET: track 80.8 -> 184.9 mm, vias 4 -> 5
- net Net-(D5-Pad2): track 10.6 -> 114.5 mm
- net /NRESET: track 0.00 -> 84.9 mm, vias 0 -> 3
- net /D6: track 195.6 -> 254.5 mm, vias 7 -> 8
- net /NBDTACK: track 4.42 -> 61.8 mm, vias 0 -> 1
- net /DIPSW3: track 12.5 -> 69.3 mm, vias 0 -> 2
- net /DIPSW2: track 16.3 -> 70.9 mm, vias 0 -> 2
- net /DIPSW4: track 15.6 -> 68.1 mm, vias 0 -> 2
- net /DIPSW5: track 19.5 -> 67.9 mm, vias 0 -> 2
- net /NBIMA: track 3.82 -> 46.7 mm
- net /DIPSW0: track 28.6 -> 71.1 mm, vias 0 -> 2
- net /TCK: track 5.41 -> 47.9 mm
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- added copper zone on B.Cu, net GND
- added copper zone on F.Cu, net GND
Other:
- net class PWR: trace_width 0.25 -> 0.8; via_dia 0.8 -> 1.2; via_drill 0.4 -> 0.8
- board text added: "+5V"
- board text added: "3.3V"
- board text added: "BA1"
- board text added: "BA10"
- board text added: "BA11"
- board text added: "BA12"
- board text added: "BA13"
- board text added: "BA14"
- board text added: "BA15"
- board text added: "BA16"
- board text added: "BA17"
- board text added: "BA18"
- board text added: "BA19"
- board text added: "BA2"
- board text added: "BA20"
- board text added: "BA21"
- board text added: "BA22"
- board text added: "BA23"
- board text added: "BA3"
- board text added: "BA4"
- board text added: "BA5"
- board text added: "BA6"
- board text added: "BA7"
- board text added: "BA8"
- board text added: "BA9"
- board text added: "BD0"
- board text added: "BD1"
- board text added: "BD10"
- board text added: "BD11"
- board text added: "BD13"
- board text added: "BD14"
- board text added: "BD15"
- board text added: "BD2"
- board text added: "BD3"
- board text added: "BD4"
- board text added: "BD6"
- board text added: "BD7"
- board text added: "BD8"
- board text added: "BD9"
- board text added: "BRNW"
- board text added: "DTACK"
- board text added: "FLASH_RY"
- board text added: "IMA"
- board text added: "NBAS"
- board text added: "NBLD"
- board text added: "NBRESET"
- board text added: "NBUD"
- board text added: "NCERAM"
- board text added: "NCEROM"
- board text added: "NOE"
- board text added: "NPS"
- board text added: "NWE"
- board text added: "OE245"
- board text added: "ROMADR0"
- board text added: "ROMADR1"
- board text added: "ROMADR2"
- board text added: "ROMADR3"
- board text added: "STM32_BUSEN"
- board text removed: "I2C and +5V"

Commit message: Layout ready.
Routing:
- added copper zone on B.Cu, net +3V3
- removed copper zone on B.Cu, net GND
Changed lines of the file:
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@@
     (polygon
       (pts
-        (xy 215.011 29.972) (xy 29.972 29.972) (xy 29.972 146.05) (xy 215.011 146.05)
+        (xy 29.972 29.972) (xy 215.011 29.972) (xy 215.011 146.05) (xy 29.972 146.05)
       )
     )
   )
-  (zone (net 2) (net_name GND) (layer B.Cu) (hatch edge 0.508)
+  (zone (net 1) (net_name +3V3) (layer B.Cu) (hatch edge 0.508)
     (connect_pads (clearance 0.508))
     (min_thickness 0.254)
